File: TSAL/TSAL.kicad_pcb (KiCad board)
At the start: 2 copper layers, 72.7 x 58.4 mm, 55 parts, among them IC1 SN74AHCT08DG4, IC2 74LVC1GU04DBVRG4, IC3 CD4002BNSR, IC4 NA555DR, IC5 SN74LVC1G27DCKR, IC6 SN74AHC1G08DBV3, J1 30700-5100, K1 ADJ-53005, U1 74LVC1G332GW-Q100H, U10 STN1HNK60, U2 LM339DT, U3 LM339DT, U4 74LVC1G332GW-Q100H, U5 SN74AHC1G02DBVRE4, U6 SI2302-NMOSFET, U7 SI2302-NMOSFET, U8 STN1HNK60

Commit message: Update TSAL.kicad_pcb
Pruebaa
Routing:
- net U2_14: track 17.3 -> 20.4 mm
Changed lines of the file:
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@@
-	)
-	(segment
-		(start 122.1391 114.3379)
-		(end 124.323 114.3379)
-		(width 0.254)
-		(layer "F.Cu")
-		(net "U2_14")
 	)
 	(segment
@@
 	)
 	(segment
-		(start 120.4632 112.662)
-		(end 122.1391 114.3379)
-		(width 0.254)
-		(layer "F.Cu")
-		(net "U2_14")
-	)
-	(segment
 		(start 124.323 114.3379)
 		(end 121.529 117.1319)
@@
 		(width 0.254)
 		(layer "F.Cu")
+		(net "U2_14")
+	)
+	(segment
+		(start 120.4632 112.662)
+		(end 120.4632 110.4781)
+		(width 0.254)
+		(layer "F.Cu")
+		(net "U2_14")
+	)
+	(segment
+		(start 120.4632 110.4781)
+		(end 124.323 114.3379)
+		(width 0.254)
+		(layer "F.Cu")

Commit message: Update TSAL.kicad_pcb
Cambio prueba
Routing:
- net RELAY_FAULT: track 44.3 -> 45.0 mm
Changed lines of the file:
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@@
 	)
 	(segment
-		(start 120.5 105)
-		(end 120.386 105.114)
+		(start 120.386 105.931)
+		(end 116.322 109.995)
+		(width 0.254)
+		(layer "F.Cu")
+		(net "RELAY_FAULT")
+	)
+	(segment
+		(start 121.529 126.505)
+		(end 122.9006 125.1334)
+		(width 0.254)
+		(layer "F.Cu")
+		(net "RELAY_FAULT")
+	)
+	(segment
+		(start 116.322 109.995)
+		(end 116.322 125.87)
 		(width 0.254)
 		(layer "F.Cu")
@@
 	)
 	(segment
+		(start 119.5 104.228)
+		(end 120.386 105.114)
+		(width 0.254)
+		(layer "F.Cu")
+		(net "RELAY_FAULT")
+	)
+	(segment
+		(start 119.5 94.752)
+		(end 119.5 104.228)
+		(width 0.254)
+		(layer "F.Cu")
+		(net "RELAY_FAULT")
+	)
+	(segment
+		(start 120.386 105.114)
+		(end 120.386 105.931)
+		(width 0.254)
+		(layer "F.Cu")
+		(net "RELAY_FAULT")
+	)
+	(segment
 		(start 122.9006 125.1334)
 		(end 122.9006 124.3612)
+		(width 0.254)
+		(layer "F.Cu")
+		(net "RELAY_FAULT")
+	)
+	(segment
+		(start 120.5 93.752)
+		(end 119.5 94.752)
 		(width 0.254)
 		(layer "F.Cu")
@@
 	)
 	(segment
-		(start 120.386 105.931)
-		(end 116.322 109.995)
-		(width 0.254)
-		(layer "F.Cu")
-		(net "RELAY_FAULT")
-	)
-	(segment
 		(start 116.957 126.505)
 		(end 121.529 126.505)
-		(width 0.254)
-		(layer "F.Cu")
-		(net "RELAY_FAULT")
-	)
-	(segment
-		(start 120.386 105.114)
-		(end 120.386 105.931)
-		(width 0.254)
-		(layer "F.Cu")
-		(net "RELAY_FAULT")
-	)
-	(segment
-		(start 120.5 93.752)
-		(end 120.5 105)
-		(width 0.254)
-		(layer "F.Cu")
-		(net "RELAY_FAULT")
-	)
-	(segment
-		(start 116.322 109.995)
-		(end 116.322 125.87)
 		(width 0.254)
 		(layer "F.Cu")
@@
 		(width 0.254)
 		(layer "F.Cu")
-		(net "RELAY_FAULT")
-	)
-	(segment
-		(start 121.529 126.505)
-		(end 122.9006 125.1334)
-		(width 0.254)
-		(layer "F.Cu")
